File: kicad_load_test_board/LoadBoard.kicad_pcb (KiCad board)
At the start: 2 copper layers, 105.2 x 147 mm, 862 parts, among them J1 CONN_01X02, J2 CONN_02X06, J3 CONN_01X10, Q1 2N7002, Q2 IRFR5505, Q3 IRFZ44N, Q4 IRFZ44N, U1 MCP4725, U2 TLC271, U3 DS18B20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

Commit message: house keeping documents
Other:
- board text added: "Licensed under CERN OHL v. 1.2"
Changed lines of the file:
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@@
   (general
     (thickness 1.6)
-    (drawings 10)
+    (drawings 11)
     (tracks 538)
     (zones 0)
@@
     )
   )
+  (gr_text "Licensed under\nCERN OHL v. 1.2" (at 129.875 171.2) (layer F.SilkS)
+    (effects (font (size 1.5 1.5) (thickness 0.3)))
+  )
   (gr_text " Part No.  301-002 Iss1.0" (at 128 176) (layer F.SilkS)
